File: photodiode/photodiode.sch (KiCad schematic (older format))
At the start: 14 parts

Commit message: Photodiode schematic development
Parts:
- added C? (x2): 18pF, symbol C_Small
- added L?: L, symbol L
- added U?: USB-MICRO-B, symbol USB-MICRO-B
- added Y?: 12MHz, symbol Crystal_Small
Connections:
- net VCC is gone; now on net +3V3: C?.1, CONN?.7 (3v3), CONN?.8 (3v3), P?.1 (P1), P?.8 (P8), R?.1
- net +3V3: now also U?.29 (VDD), U?.6 (VDD), U?.1 (VBUS)
- net GND: now also J?.3 (Pin_3), U?.33 (VSS), U?.~ (SOCKET2c), C?.2, C?.2, L?.2, U?.5 (GND)
- net at U?.4 (XTALIN): now also C?.1, Y?.2
- net at U?.5 (XTALOUT): now also C?.1, Y?.1
- net PWR1+v renamed +15V
- removed net PWR1-v: J?.3 (Pin_3), U?.~ (SOCKET2c)
- net PWR2: no longer names the net of J?.2 (Pin_2)
- net PWR2: no longer U?.~ (SOCKET2c)
- new net: L?.1, U?.6 (SHELL4)
- no-connect marks 11 -> 14
Other:
- note added: "USB"
- moved on the sheet: D?, J?, U?

Commit message: Schematic complete
Parts:
- removed J?: Conn_01x02, symbol Conn_01x02
- removed L?: L, symbol L
- removed U?: USB-MICRO-B, symbol USB-MICRO-B
- added C? (x3): 100n, symbol C_Small
- added C?: 100nF, symbol C_Small
- added D?: BAS40-05, TO_SOT_Packages_SMD:SOT-23, symbol BAS40-05
- added D?: LED, symbol LED
- added J? (x2): Conn_01x16, symbol Conn_01x16
- added JP?: Jumper_NC_Small, Connectors:PINHEAD1-2, symbol Jumper_NC_Small
- added JP? (x2): JP1, Connectors:PINHEAD1-2, symbol Jumper_NC_Small
- added R?: 22k, symbol R_Small
- added R?: 1k, symbol R_Small
- added U?: LT1129-3.3_SOT223, TO_SOT_Packages_SMD:SOT-223-3Lead_TabPin2, symbol LT1129-3.3_SOT223
Connections:
- net OUT1a is gone; now on net GND: U?.~ (SOCKET2c)
- net OUT1b is gone; now on net GND: U?.~ (SOCKET2c)
- net +3V3: now also C?.1, C?.1, J?.4 (Pin_4), R?.1, R?.2, U?.3 (VO)
- net CE: now also U?.8 (PIO0_2/SSEL0/CT16B0_CAP0)
- net CLK: now also U?.15 (PIO0_6/SCK0)
- net GND: now also C?.2, C?.2, C?.2, C?.2, J?.2 (Pin_2), J?.3 (Pin_3), U?.2 (GND)
- net LED: now also U?.28 (PIO3_2), D?.1 (K)
- net RESET: now also J?.16 (Pin_16), R?.1
- net UART_RX: now also JP?.1; no longer U?.31 (PIO1_6/RXD/CT32B0_MAT0)
- net UART_TX: now also JP?.1; no longer U?.32 (PIO1_7/TXD/CT32B0_MAT1)
- net ADCin0: now reaches U?.21 (R/PIO0_11/AD0/CT32B0_MAT3)
- net ADCin0: now also U?.~ (SOCKET2c)
- net ADCin1: now reaches U?.22 (R/PIO1_0/AD1/CT32B1_CAP0)
- net ADCin1: now also U?.~ (SOCKET2c)
- new net: JP?.2, U?.31 (PIO1_6/RXD/CT32B0_MAT0)
- new net: JP?.2, U?.32 (PIO1_7/TXD/CT32B0_MAT1)
- new net: C?.1, C?.1, D?.3 (K1K2), U?.1 (VI)
- new net: D?.2 (A), R?.2
- new net +5V: D?.1 (A1), D?.2 (A2), J?.1 (Pin_1), JP?.1, JP?.2
- no-connect marks 14 -> 13
Other:
- note added: "3v3 voltage regulator"
- note removed: "USB"
- moved on the sheet: C?, U?, Y?
